File: schematics/odometer_project-DESKTOP-8EVBIF8.sch (KiCad schematic (older format))
At the start: 16 parts, among them J1 Conn_01x03_Female, J2 Conn_01x03_Female, J3 Conn_02x10_Odd_Even, J4 Conn_02x10_Odd_Even, U1 SN74HC14N

Commit message: production build
Connections:
- wire segments 107 -> 110
- no-connect marks 0 -> 24
Other:
- moved on the sheet: R3
Changed lines of the file:
@@
 EESchema Schematic File Version 4
-LIBS:odometer_project-cache
 EELAYER 30 0
 EELAYER END
@@
 F 3 "" H 10200 2000 50  0001 C CNN
 	1    10200 2000
-	0    1    1    0
+	1    0    0    -1
 $EndComp
 Text GLabel 8700 1700 0    50   Input ~ 0
@@
 	9600 2000 9700 2000
 Wire Wire Line
-	10000 2000 10200 2000
+	10050 2000 10200 2000
 Wire Wire Line
 	9600 2100 9700 2100
@@
 L Device:R R3
 U 1 1 5F77198D
-P 9850 2000
-F 0 "R3" H 9920 2046 50  0000 L CNN
-F 1 "330" H 9920 1955 50  0000 L CNN
-F 2 "Resistor_SMD:R_0805_2012Metric_Pad1.15x1.40mm_HandSolder" V 9780 2000 50  0001 C CNN
-F 3 "~" H 9850 2000 50  0001 C CNN
-F 4 "C17630" H 9850 2000 50  0001 C CNN "LCSC Part #"
-	1    9850 2000
+P 9900 2000
+F 0 "R3" H 9970 2046 50  0000 L CNN
+F 1 "330" H 9970 1955 50  0000 L CNN
+F 2 "Resistor_SMD:R_0805_2012Metric_Pad1.15x1.40mm_HandSolder" V 9830 2000 50  0001 C CNN
+F 3 "~" H 9900 2000 50  0001 C CNN
+F 4 "C17630" H 9900 2000 50  0001 C CNN "LCSC Part #"
+	1    9900 2000
 	0    1    1    0
 $EndComp
@@
 $EndComp
 Wire Wire Line
-	1700 2100 1700 2000
-Wire Wire Line
-	1600 4100 1600 4250
-Wire Wire Line
 	2400 3100 2300 3100
 Wire Wire Line
@@
 Wire Wire Line
 	2300 2500 2400 2500
-Wire Notes Line
-	4200 550  4200 7750
 $Comp
 L power:+5V #PWR0116
@@
 Wire Wire Line
 	8300 1800 8800 1800
+NoConn ~ 8800 2200
+NoConn ~ 8800 2300
+NoConn ~ 8800 2400
+NoConn ~ 8800 2500
+NoConn ~ 2300 3600
+NoConn ~ 2300 3700
+NoConn ~ 1900 4100
+NoConn ~ 1700 4100
+NoConn ~ 1300 3700
+NoConn ~ 1300 3600
+NoConn ~ 1300 3300
+NoConn ~ 1300 3100
+NoConn ~ 1300 3000
+NoConn ~ 1300 2900
+NoConn ~ 1300 2800
+NoConn ~ 1300 2500
+NoConn ~ 1300 2400
+NoConn ~ 3000 6200
+NoConn ~ 3000 6300
+NoConn ~ 3000 6400
+NoConn ~ 2400 6400
+NoConn ~ 2400 6300
+NoConn ~ 2400 6200
+NoConn ~ 2300 2400
+Wire Wire Line
+	1700 2000 1700 2100
+Wire Wire Line
+	1600 4100 1600 4250
+$Comp
+L power:PWR_FLAG #FLG0102
+U 1 1 5F8A9181
+P 9700 2000
+F 0 "#FLG0102" H 9700 2075 50  0001 C CNN
+F 1 "PWR_FLAG" H 9700 2173 50  0000 C CNN
+F 2 "" H 9700 2000 50  0001 C CNN
+F 3 "~" H 9700 2000 50  0001 C CNN
+	1    9700 2000
+	1    0    0    -1
+$EndComp
+Connection ~ 9700 2000
+Wire Wire Line
+	9700 2000 9750 2000
+Wire Wire Line
+	5400 7000 5400 6950
+Wire Wire Line
+	5450 7000 5400 7000
+$Comp
+L power:GND #PWR0125
+U 1 1 5F88F13E
+P 5400 6950
+F 0 "#PWR0125" H 5400 6700 50  0001 C CNN
+F 1 "GND" H 5405 6777 50  0000 C CNN
+F 2 "" H 5400 6950 50  0001 C CNN
+F 3 "" H 5400 6950 50  0001 C CNN
+	1    5400 6950
+	-1   0    0    1
+$EndComp
+$Comp
+L power:PWR_FLAG #FLG0101
+U 1 1 5F88EF1C
+P 5450 7000
+F 0 "#FLG0101" H 5450 7075 50  0001 C CNN
+F 1 "PWR_FLAG" V 5450 7128 50  0000 L CNN
+F 2 "" H 5450 7000 50  0001 C CNN
+F 3 "~" H 5450 7000 50  0001 C CNN
+	1    5450 7000
+	0    1    1    0
+$EndComp
+Wire Notes Line
+	4200 550  4200 7750
 $EndSCHEMATC
