File: schematics/odometer_project.kicad_pcb (KiCad board)
At the start: 2 copper layers, 96.5 x 76.2 mm, 32 parts, among them J2 Conn_01x03_Female, J3 Conn_02x10_Odd_Even, J4 Conn_02x10_Odd_Even, SW1 SW_SPST, SW2 SW_SPST, SW3 SW_SPST, U1 SN74HC14N

Commit message: fixed lcd pin connections and xtra halls
Parts:
- removed G***: LOGO, meme_library:little_creatures
- removed G***: LOGO, meme_library:pepe_frog
- removed REF** (x4): MountingHole_3mm_Pad_Via, MountingHole:MountingHole_3mm_Pad_Via
- added D4: LED_Yellow, LED_SMD:LED_0805_2012Metric_Pad1.15x1.40mm_HandSolder, F.Cu at (269.0, 125.5)
- added D5: LED_Yellow, LED_SMD:LED_0805_2012Metric_Pad1.15x1.40mm_HandSolder, F.Cu at (189.0, 125.7)
- added J1: Conn_01x03_Female, Connector_PinHeader_2.54mm:PinHeader_1x03_P2.54mm_Horizontal, F.Cu at (185.9, 125.0)
- added JP1: Jumper_3_Open, Connector_PinHeader_2.54mm:PinHeader_1x03_P2.54mm_Vertical, F.Cu at (243.3, 130.6)
- added JP2: Jumper_3_Open, Connector_PinHeader_2.54mm:PinHeader_1x03_P2.54mm_Vertical, F.Cu at (222.2, 133.6)
- added R11: 330, Resistor_SMD:R_0805_2012Metric_Pad1.15x1.40mm_HandSolder, F.Cu at (266.7, 125.5)
- added R12: 330, Resistor_SMD:R_0805_2012Metric_Pad1.15x1.40mm_HandSolder, F.Cu at (191.0, 125.7)
- added RV1: R_POT, Potentiometer_THT:Potentiometer_Bourns_3296W_Vertical, F.Cu at (255.8, 125.7)
Connections:
- net /sheet5F7CC05F/vout renamed /sw2/vout
- net /sheet5F7CF7B9/vout renamed /sw3/vout
- net Net-(A1-Pad6) renamed hall1
- A1 pad 1: Net-(A1-Pad1) -> (no net)
- A1 pad 12: lcd_rw -> Net-(A1-Pad12)
- A1 pad 16: Net-(A1-Pad16) -> (no net)
- A1 pad 17: Net-(A1-Pad17) -> (no net)
- A1 pad 18: Net-(A1-Pad18) -> (no net)
- A1 pad 19: Net-(A1-Pad19) -> (no net)
- A1 pad 2: Net-(A1-Pad2) -> (no net)
- A1 pad 20: Net-(A1-Pad20) -> (no net)
- A1 pad 21: Net-(A1-Pad21) -> (no net)
- A1 pad 22: Net-(A1-Pad22) -> (no net)
- A1 pad 25: Net-(A1-Pad25) -> (no net)
- A1 pad 26: Net-(A1-Pad26) -> (no net)
- A1 pad 28: Net-(A1-Pad28) -> (no net)
- A1 pad 29: GND -> lcd_rw
- A1 pad 3: Net-(A1-Pad3) -> (no net)
- A1 pad 30: Net-(A1-Pad30) -> (no net)
- A1 pad 4: Net-(A1-Pad4) -> lcd_rw
- A1 pad 5: soft_reset -> Net-(A1-Pad5)
- C1 pad 2: GND -> lcd_rw
- C2 pad 2: GND -> lcd_rw
- C3 pad 2: GND -> lcd_rw
- C4 pad 2: GND -> lcd_rw
- D1 pad 1: GND -> lcd_rw
- D2 pad 1: GND -> lcd_rw
- D3 pad 1: GND -> lcd_rw
- DS1 pad 1: GND -> lcd_rw
- DS1 pad 10: lcd_bit4 -> (no net)
- DS1 pad 11: Net-(DS1-Pad11) -> lcd_bit1
- DS1 pad 12: Net-(DS1-Pad12) -> lcd_bit2
- DS1 pad 13: Net-(DS1-Pad13) -> lcd_bit3
- DS1 pad 14: Net-(DS1-Pad14) -> lcd_bit4
- DS1 pad 16: GND -> lcd_rw
- DS1 pad 7: lcd_bit1 -> (no net)
- DS1 pad 8: lcd_bit2 -> (no net)
- DS1 pad 9: lcd_bit3 -> (no net)
- J2 pad 3: GND -> lcd_rw
- J4 pad 10: GND -> lcd_rw
- J4 pad 12: GND -> lcd_rw
- J4 pad 14: GND -> lcd_rw
- J4 pad 16: GND -> lcd_rw
- J4 pad 18: GND -> lcd_rw
- J4 pad 2: GND -> lcd_rw
- J4 pad 20: GND -> lcd_rw
- J4 pad 4: GND -> lcd_rw
- J4 pad 6: GND -> lcd_rw
- J4 pad 8: GND -> lcd_rw
- SW1 pad 2: GND -> lcd_rw
- SW2 pad 2: GND -> lcd_rw
- SW3 pad 2: GND -> lcd_rw
- U1 pad 10: Net-(U1-Pad10) -> (no net)
- U1 pad 11: Net-(U1-Pad11) -> (no net)
- U1 pad 12: Net-(U1-Pad12) -> (no net)
- U1 pad 13: Net-(U1-Pad13) -> (no net)
- U1 pad 7: GND -> lcd_rw
- U1 pad 8: Net-(U1-Pad8) -> (no net)
- U1 pad 9: Net-(U1-Pad9) -> (no net)
Routing:
- net lcd_rw: track 72.2 -> 5.83 mm, vias 0 -> 10
- net Net-(A1-Pad12): track 0.00 -> 65.2 mm
- net Net-(A1-Pad5): track 0.00 -> 54.5 mm, vias 0 -> 2
- net hall2: track 0.00 -> 48.4 mm
- net Net-(DS1-Pad3): track 0.00 -> 15.8 mm
- net soft_reset: track 55.8 -> 63.4 mm
- net lcd_bit1: track 64.1 -> 56.7 mm
- net lcd_bit2: track 65.3 -> 60.1 mm
- net Net-(D4-Pad2): track 0.00 -> 3.13 mm
- net lcd_bit3: track 68.0 -> 64.9 mm
- net lcd_enable: track 71.1 -> 74.0 mm
- net Net-(D5-Pad2): track 0.00 -> 2.89 mm
- net hall1: track 48.2 -> 49.9 mm, vias 0 -> 1
- net lcd_bit4: track 71.4 -> 69.9 mm
- net lcd_rs: track 74.5 -> 75.3 mm
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- added copper zone on B.Cu, net lcd_rw
- removed copper zone on B.Cu, net GND
Other:
- board text added: "Odometer V.2.1"
- board text added: "hall1"
- board text added: "hall2"
- board text added: "hall2 | rst"
- board text added: "inacc | stdio"
- board text added: "int1"
- board text added: "int_selection"
- board text added: "rst_selection"
- board text removed: "Odometer V.2.0"
- board text removed: "rst"

Commit message: added schematic notes
Parts:
- added G***: LOGO, meme_lib:brrr, B.Cu at (194.3, 129.3)
- added REF**: MountingHole_3.2mm_M3_Pad_Via, MountingHole:MountingHole_3.2mm_M3_Pad_Via, F.Cu at (262.4, 112.0)
- added REF**: MountingHole_3.2mm_M3_Pad_Via, MountingHole:MountingHole_3.2mm_M3_Pad_Via, F.Cu at (186.6, 134.4)
- added REF**: MountingHole_3.2mm_M3_Pad_Via, MountingHole:MountingHole_3.2mm_M3_Pad_Via, F.Cu at (192.5, 94.2)
