File: schematics/switch_debounced.sch (KiCad schematic (older format))
At the start: 6 parts, among them SW1 SW_SPST

Commit message: production build
Changed lines of the file:
@@
 EESchema Schematic File Version 4
+LIBS:odometer_project-cache
 EELAYER 30 0
 EELAYER END
@@
 AR Path="/5F7CC063/5F7A2F6B" Ref="SW2"  Part="1"
 AR Path="/5F7CF7BD/5F7A2F6B" Ref="SW3"  Part="1"
-F 0 "SW1" V 4654 4048 50  0000 L CNN
+F 0 "SW3" V 4654 4048 50  0000 L CNN
 F 1 "SW_SPST" V 4745 4048 50  0000 L CNN
 F 2 "Button_Switch_THT:SW_PUSH_6mm_H4.3mm" H 4700 3950 50  0001 C CNN
@@
 AR Path="/5F7CC063/5F7A3360" Ref="#PWR0106"  Part="1"
 AR Path="/5F7CF7BD/5F7A3360" Ref="#PWR0113"  Part="1"
-F 0 "#PWR0101" H 4700 4250 50  0001 C CNN
+F 0 "#PWR0113" H 4700 4250 50  0001 C CNN
 F 1 "GND" H 4705 4327 50  0000 C CNN
 F 2 "" H 4700 4500 50  0001 C CNN
@@
 AR Path="/5F7CC063/5F7A3875" Ref="#PWR0107"  Part="1"
 AR Path="/5F7CF7BD/5F7A3875" Ref="#PWR0114"  Part="1"
-F 0 "#PWR0102" H 4700 2500 50  0001 C CNN
+F 0 "#PWR0114" H 4700 2500 50  0001 C CNN
 F 1 "+5V" H 4715 2823 50  0000 C CNN
 F 2 "" H 4700 2650 50  0001 C CNN
@@
 AR Path="/5F7CC063/5F7A4488" Ref="R4"  Part="1"
 AR Path="/5F7CF7BD/5F7A4488" Ref="R6"  Part="1"
-F 0 "R1" H 4770 3046 50  0000 L CNN
+F 0 "R6" H 4770 3046 50  0000 L CNN
 F 1 "10K" H 4770 2955 50  0000 L CNN
 F 2 "Resistor_SMD:R_0805_2012Metric_Pad1.15x1.40mm_HandSolder" V 4630 3000 50  0001 C CNN
@@
 AR Path="/5F7CC063/5F7A534F" Ref="C3"  Part="1"
 AR Path="/5F7CF7BD/5F7A534F" Ref="C4"  Part="1"
-F 0 "C2" H 5565 3996 50  0000 L CNN
+F 0 "C4" H 5565 3996 50  0000 L CNN
 F 1 "0.1uF" H 5565 3905 50  0000 L CNN
 F 2 "Capacitor_SMD:C_0805_2012Metric_Pad1.15x1.40mm_HandSolder" H 5488 3800 50  0001 C CNN
@@
 AR Path="/5F7CC063/5F7A59C8" Ref="#PWR0112"  Part="1"
 AR Path="/5F7CF7BD/5F7A59C8" Ref="#PWR0115"  Part="1"
-F 0 "#PWR0105" H 5450 4250 50  0001 C CNN
+F 0 "#PWR0115" H 5450 4250 50  0001 C CNN
 F 1 "GND" H 5455 4327 50  0000 C CNN
 F 2 "" H 5450 4500 50  0001 C CNN
@@
 AR Path="/5F7CC063/5F7D50A7" Ref="R5"  Part="1"
 AR Path="/5F7CF7BD/5F7D50A7" Ref="R7"  Part="1"
-F 0 "R2" H 5170 3446 50  0000 L CNN
+F 0 "R7" H 5170 3446 50  0000 L CNN
 F 1 "10K" H 5170 3355 50  0000 L CNN
 F 2 "Resistor_SMD:R_0805_2012Metric_Pad1.15x1.40mm_HandSolder" V 5030 3400 50  0001 C CNN
@@
 AR Path="/5F7CC063/5F8214CD" Ref="D2"  Part="1"
 AR Path="/5F7CF7BD/5F8214CD" Ref="D3"  Part="1"
-F 0 "D1" V 6139 4033 50  0000 R CNN
+F 0 "D3" V 6139 4033 50  0000 R CNN
 F 1 "LED_Yellow" V 6048 4033 50  0000 R CNN
 F 2 "LED_SMD:LED_0805_2012Metric_Pad1.15x1.40mm_HandSolder" H 6100 4150 50  0001 C CNN
@@
 AR Path="/5F7CC063/5F8223FC" Ref="R9"  Part="1"
 AR Path="/5F7CF7BD/5F8223FC" Ref="R10"  Part="1"
-F 0 "R8" H 6031 3704 50  0000 R CNN
+F 0 "R10" H 6031 3704 50  0000 R CNN
 F 1 "330" H 6031 3795 50  0000 R CNN
 F 2 "Resistor_SMD:R_0805_2012Metric_Pad1.15x1.40mm_HandSolder" V 6030 3750 50  0001 C CNN
@@
 AR Path="/5F7CC063/5F8242EB" Ref="#PWR04"  Part="1"
 AR Path="/5F7CF7BD/5F8242EB" Ref="#PWR05"  Part="1"
-F 0 "#PWR03" H 6100 4250 50  0001 C CNN
+F 0 "#PWR05" H 6100 4250 50  0001 C CNN
 F 1 "GND" H 6105 4327 50  0000 C CNN
 F 2 "" H 6100 4500 50  0001 C CNN
